Commit message: add drvie system so it can be operated by keyboard and fixing the wheel rotation

File: urdf/robot.urdf (robot description, URDF)
Before this commit: robot challenge_rover, 13 links, 12 joints
Joints:
- joint fl_joint: axis 0 0 1 -> 0 0 -1
- joint fr_joint: axis 0 0 1 -> 0 0 -1
- joint rl_joint: axis 0 0 1 -> 0 0 -1
- joint rr_joint: axis 0 0 1 -> 0 0 -1

Commit message: Adding for Task 2

File: urdf/robot.urdf (robot description, URDF)
Before this commit: robot challenge_rover, 13 links, 12 joints
Links:
- added link base_footprint
- link imu_link: mass None -> 0.1
Joints:
- added joint base_footprint_joint: type fixed, parent base_footprint, child base_link, origin xyz=0 0 0 rpy=0 0 0
